File: pcb/Microcontroller.kicad_sch (KiCad schematic)
At the start: 18 parts, among them U1 STM32F405RGTx, Y1 8MHz

Commit message: feat: working changes
Parts:
- removed R3: 1MΩ, Resistor_SMD:R_0603_1608Metric, symbol Device:R
- removed Y1: 8MHz, Crystal:Crystal_SMD_3225-4Pin_3.2x2.5mm, symbol Device:Crystal
- added Y1: FA-238_16.0000MA20W-C, prometheus-65-footprints:FA-238_16.0000MA20W-C, symbol prometheus-65-symbols:FA-238_16.0000MA20W-C
- renumbered C7 to C10, C8 to C11, C9 to C12, C10 to C13, C11 to C14, C12 to C15, C13 to C16, C1 to C4, C2 to C5, C3 to C6, C4 to C7, C5 to C8, C6 to C9, R1 to R34, R2 to R35, U1 to U4
Connections:
- net GND: now also Y1.2 (GND), Y1.4 (GND)
- net MUX_A0: now also U4.8 (PC0); no longer U4.2 (PC13)
- net MUX_A1: now also U4.9 (PC1); no longer U4.3 (PC14)
- net MUX_EN1: now reaches U4.10 (PC2)
- net MUX_EN2: now reaches U4.11 (PC3)
- net MUX_EN3: now reaches U4.24 (PC4)
- net at C12.2, U4.5 (PH0): now also Y1.1
- net at C13.2, U4.6 (PH1): now also Y1.3
- net MUX_A2: no longer names the net of U4.4 (PC15)
- net MUX_D0 renamed MUX_C0
- net MUX_D1 renamed MUX_C1
- net MUX_D2 renamed MUX_C2
- net MUX_D3 renamed MUX_C3
- net MUX_D4 renamed MUX_C4
- net MUX_D5 renamed MUX_C5
- net MUX_D6 renamed MUX_C6
- net MUX_D7: no longer names the net of U4.23 (PA7)
- no-connect marks 30 -> 29
Other:
- moved on the sheet: C12, C13
