File: pcb/Multiplexer.kicad_sch (KiCad schematic)
At the start: 1 part, among them U5 TMUX1308

Commit message: feat: working changes
Parts:
- removed U5: TMUX1308, prometheus-65-footprints:TMUX1308BQBR, symbol prometheus-65-symbols:TMUX1308
- added C23: 100nF, symbol Device:C
- added U7: TMUX1109RSVR, prometheus-65-footprints:TMUX1109RSVR, symbol prometheus-65-symbols:TMUX1109RSVR
- added U8, U9: TPD4E05U06DQAR, prometheus-65-footprints:TPD4E05U06DQAR, symbol prometheus-65-symbols:TPD4E05U06DQAR
Connections:
- net +3.3VD: now also C23.1
- net GND: now also U7.1 (VSS), U7.13 (GND), U8.3 (GND), U8.8 (GND), U9.3 (GND), U9.8 (GND)
- net MUX_A0: now also U7.15 (A0)
- net MUX_A1: now also U7.14 (A1)
- new net: C23.2, U7.12 (VDD)
- new net MUX_DA: U7.6 (DA)
- new net MUX_DB: U7.7 (DB)
- new net MUX_EN: U7.16 (EN)
- new net SIG_1A: U7.2 (S1A), U8.1 (D1+)
- new net SIG_1B: U7.11 (S1B), U9.1 (D1+)
- new net SIG_2A: U7.3 (S2A), U8.2 (D1-)
- new net SIG_2B: U7.10 (S2B), U9.4 (D2+)
- new net SIG_3A: U7.4 (S3A), U8.4 (D2+)
- new net SIG_3B: U7.9 (S3B), U9.2 (D1-)
- new net SIG_4A: U7.5 (S4A), U8.5 (D2-)
- new net SIG_4B: U7.8 (S4B), U9.5 (D2-)
- no-connect marks 0 -> 8
