File: pcb/prometheus-65.kicad_pcb (KiCad board)
At the start: 4 copper layers, 424 parts, among them J1 Conn_01x04_Socket, SW1 RotaryEncoder_Switch, U1 STM32F405RGTx, U10 TMR2652D, U11 TMR2652D, U12 TMR2652D, U13 TMR2652D, U14 TMR2652D, U15 TMR2652D, U16 TMR2652D, U17 TMR2652D, U18 TMR2652D, U19 TMR2652D, U2 TPS7A4700, U20 TMR2652D, U21 TMUX1308, U22 TMR2652D, U23 TMR2652D, U24 TMR2652D, U25 TMR2652D, U26 TMR2652D, U27 TMR2652D, U28 TMR2652D, U29 TMR2652D, U3 TPS7A4700, U30 TMUX1308, U31 TMR2652D, U32 TMR2652D, U33 TMR2652D, U34 TMR2652D, U35 TMR2652D, U36 TMR2652D, U37 TMR2652D, U38 TMR2652D, U39 TMUX1308, U4 TMR2652D, U40 TMR2652D, U41 TMR2652D, U42 TMR2652D, U43 TMR2652D, U44 TMR2652D, U45 TMR2652D, U46 TMR2652D, U47 TMR2652D, U48 TMR2652D, U49 TMR2652D, U5 TMUX1308, U50 TMR2652D, U51 TMR2652D, U52 TMR2652D, U53 TMR2652D, U54 TMR2652D, U55 TMR2652D, U56 TMR2652D, U57 TMR2652D, U58 TMR2652D, U59 TMR2652D, U6 TMR2652D, U60 TMR2652D, U61 TMR2652D, U62 TMR2652D, U63 TMR2652D, U64 TMR2652D, U65 TMR2652D, U66 TMR2652D, U67 TMR2652D, U68 TMR2652D, U69 TMR2652D, U7 TMR2652D, U70 TMR2652D, U71 TMR2652D, U72 TMUX1308, U73 TMUX1308, U74 TMUX1308, U75 TMUX1308, U76 74AHCT125, U8 TMR2652D, U9 TMR2652D, Y1 8MHz

Commit message: feat: completed layout for a single switch
Parts:
- removed C100, C102, C104, C106, C108, C110, C112, C114, C116, C118, C120, C122, C124, C126, C128, C130, C132, C134, C136, C138, C140, C142, C144, C146, C84, C86, C88, C90, C92, C94, C96, C98: 0.1uF, Capacitor_SMD:C_0402_1005Metric
- removed C101, C103, C105, C107, C109, C111, C113, C115, C117, C119, C121, C123, C125, C127, C129, C131, C133, C135, C137, C139, C141, C143, C145, C147, C85, C87, C89, C91, C93, C95, C97, C99: 20pF, Capacitor_SMD:C_0402_1005Metric
- removed D10, D11, D12, D13, D14, D15, D16, D17, D18, D19, D2, D20, D21, D22, D23, D24, D25, D26, D27, D28, D29, D3, D30, D31, D32, D33, D34, D35, D36, D37, D38, D39, D4, D40, D41, D42, D43, D44, D45, D46, D47, D48, D49, D5, D50, D51, D52, D53, D54, D55, D56, D57, D58, D59, D6, D60, D61, D62, D63, D64, D7, D8, D9: SK6812MINI, LED_SMD:LED_SK6812MINI_PLCC4_3.5x3.5mm_P1.75mm
- removed U21, U30, U39, U5, U72, U73, U74, U75: TMUX1308, prometheus-65-footprints:TMUX1308BQBR
- added LED10: SK6812MINI-E, PCM_marbastlib-various:LED_6028R, B.Cu at (-58.3, 59.7)
- added LED11: SK6812MINI-E, PCM_marbastlib-various:LED_6028R, B.Cu at (-65.1, 18.7)
- added LED12: SK6812MINI-E, PCM_marbastlib-various:LED_6028R, B.Cu at (-65.1, 23.8)
- added LED13: SK6812MINI-E, PCM_marbastlib-various:LED_6028R, B.Cu at (-65.1, 28.9)
- added LED14: SK6812MINI-E, PCM_marbastlib-various:LED_6028R, B.Cu at (-65.1, 34.1)
- added LED15: SK6812MINI-E, PCM_marbastlib-various:LED_6028R, B.Cu at (-65.1, 39.2)
- added LED16: SK6812MINI-E, PCM_marbastlib-various:LED_6028R, B.Cu at (-65.1, 44.3)
- added LED17: SK6812MINI-E, PCM_marbastlib-various:LED_6028R, B.Cu at (-65.1, 49.4)
- added LED18: SK6812MINI-E, PCM_marbastlib-various:LED_6028R, B.Cu at (-65.1, 54.5)
- added LED19: SK6812MINI-E, PCM_marbastlib-various:LED_6028R, B.Cu at (-65.1, 59.7)
- added LED2: SK6812MINI-E, PCM_marbastlib-various:LED_6028R, B.Cu at (-58.3, 18.7)
- added LED20: SK6812MINI-E, PCM_marbastlib-various:LED_6028R, B.Cu at (-71.8, 18.7)
- added LED21: SK6812MINI-E, PCM_marbastlib-various:LED_6028R, B.Cu at (-71.8, 23.8)
- added LED22: SK6812MINI-E, PCM_marbastlib-various:LED_6028R, B.Cu at (-71.8, 28.9)
- added LED23: SK6812MINI-E, PCM_marbastlib-various:LED_6028R, B.Cu at (-71.8, 34.1)
- added LED24: SK6812MINI-E, PCM_marbastlib-various:LED_6028R, B.Cu at (-71.8, 39.2)
- added LED25: SK6812MINI-E, PCM_marbastlib-various:LED_6028R, B.Cu at (-71.8, 44.3)
- added LED26: SK6812MINI-E, PCM_marbastlib-various:LED_6028R, B.Cu at (-71.8, 49.4)
- added LED27: SK6812MINI-E, PCM_marbastlib-various:LED_6028R, B.Cu at (-71.8, 54.5)
- added LED28: SK6812MINI-E, PCM_marbastlib-various:LED_6028R, B.Cu at (-71.8, 59.7)
- added LED29: SK6812MINI-E, PCM_marbastlib-various:LED_6028R, B.Cu at (-78.5, 18.7)
- added LED3: SK6812MINI-E, PCM_marbastlib-various:LED_6028R, B.Cu at (-58.3, 23.8)
- added LED30: SK6812MINI-E, PCM_marbastlib-various:LED_6028R, B.Cu at (-78.5, 23.8)
- added LED31: SK6812MINI-E, PCM_marbastlib-various:LED_6028R, B.Cu at (-78.5, 28.9)
- added LED32: SK6812MINI-E, PCM_marbastlib-various:LED_6028R, B.Cu at (-78.5, 34.1)
- added LED33: SK6812MINI-E, PCM_marbastlib-various:LED_6028R, B.Cu at (-78.5, 39.2)
- added LED34: SK6812MINI-E, PCM_marbastlib-various:LED_6028R, B.Cu at (-78.5, 44.3)
- added LED35: SK6812MINI-E, PCM_marbastlib-various:LED_6028R, B.Cu at (-78.5, 49.4)
- added LED36: SK6812MINI-E, PCM_marbastlib-various:LED_6028R, B.Cu at (-78.5, 54.5)
- added LED37: SK6812MINI-E, PCM_marbastlib-various:LED_6028R, B.Cu at (-78.5, 59.7)
- added LED38: SK6812MINI-E, PCM_marbastlib-various:LED_6028R, B.Cu at (-85.2, 18.7)
- added LED39: SK6812MINI-E, PCM_marbastlib-various:LED_6028R, B.Cu at (-85.2, 23.8)
- added LED4: SK6812MINI-E, PCM_marbastlib-various:LED_6028R, B.Cu at (-58.3, 28.9)
- added LED40: SK6812MINI-E, PCM_marbastlib-various:LED_6028R, B.Cu at (-85.2, 28.9)
- added LED41: SK6812MINI-E, PCM_marbastlib-various:LED_6028R, B.Cu at (-85.2, 34.1)
- added LED42: SK6812MINI-E, PCM_marbastlib-various:LED_6028R, B.Cu at (-85.2, 39.2)
- added LED43: SK6812MINI-E, PCM_marbastlib-various:LED_6028R, B.Cu at (-85.2, 44.3)
- added LED44: SK6812MINI-E, PCM_marbastlib-various:LED_6028R, B.Cu at (-85.2, 49.4)
- added LED45: SK6812MINI-E, PCM_marbastlib-various:LED_6028R, B.Cu at (-85.2, 54.5)
- added LED46: SK6812MINI-E, PCM_marbastlib-various:LED_6028R, B.Cu at (-85.2, 59.7)
- added LED47: SK6812MINI-E, PCM_marbastlib-various:LED_6028R, B.Cu at (-91.9, 18.7)
- added LED48: SK6812MINI-E, PCM_marbastlib-various:LED_6028R, B.Cu at (-91.9, 23.8)
- added LED49: SK6812MINI-E, PCM_marbastlib-various:LED_6028R, B.Cu at (-91.9, 28.9)
- added LED5: SK6812MINI-E, PCM_marbastlib-various:LED_6028R, B.Cu at (-58.3, 34.1)
- added LED50: SK6812MINI-E, PCM_marbastlib-various:LED_6028R, B.Cu at (-91.9, 34.1)
- added LED51: SK6812MINI-E, PCM_marbastlib-various:LED_6028R, B.Cu at (-91.9, 39.2)
- added LED52: SK6812MINI-E, PCM_marbastlib-various:LED_6028R, B.Cu at (-91.9, 44.3)
- added LED53: SK6812MINI-E, PCM_marbastlib-various:LED_6028R, B.Cu at (-91.9, 49.4)
- added LED54: SK6812MINI-E, PCM_marbastlib-various:LED_6028R, B.Cu at (-91.9, 54.5)
- added LED55: SK6812MINI-E, PCM_marbastlib-various:LED_6028R, B.Cu at (-91.9, 59.7)
- added LED56: SK6812MINI-E, PCM_marbastlib-various:LED_6028R, B.Cu at (-98.7, 18.7)
- added LED57: SK6812MINI-E, PCM_marbastlib-various:LED_6028R, B.Cu at (-98.7, 23.8)
- added LED58: SK6812MINI-E, PCM_marbastlib-various:LED_6028R, B.Cu at (-98.7, 28.9)
- added LED59: SK6812MINI-E, PCM_marbastlib-various:LED_6028R, B.Cu at (-98.7, 34.1)
- added LED6: SK6812MINI-E, PCM_marbastlib-various:LED_6028R, B.Cu at (-58.3, 39.2)
- added LED60: SK6812MINI-E, PCM_marbastlib-various:LED_6028R, B.Cu at (-98.7, 39.2)
- added LED61: SK6812MINI-E, PCM_marbastlib-various:LED_6028R, B.Cu at (-98.7, 44.3)
- added LED62: SK6812MINI-E, PCM_marbastlib-various:LED_6028R, B.Cu at (-98.7, 49.4)
- added LED63: SK6812MINI-E, PCM_marbastlib-various:LED_6028R, B.Cu at (-98.7, 54.5)
- added LED64: SK6812MINI-E, PCM_marbastlib-various:LED_6028R, B.Cu at (-98.7, 59.7)
- added LED7: SK6812MINI-E, PCM_marbastlib-various:LED_6028R, B.Cu at (-58.3, 44.3)
- added LED8: SK6812MINI-E, PCM_marbastlib-various:LED_6028R, B.Cu at (-58.3, 49.4)
- added LED9: SK6812MINI-E, PCM_marbastlib-various:LED_6028R, B.Cu at (-58.3, 54.5)
- C1, C11, C12, C13, C14, C15, C16, C17, C18, C19, C2, C22, C24, C26, C28, C3, C30, C32, C34, C36, C38, C4, C40, C42, C44, C46, C48, C5, C50, C52, C54, C56, C58, C6, C60, C62, C64, C66, C68, C7, C70, C72, C74, C76, C78, C8, C80, C82, J1, R1, R10, R11, R12, R13, R14, R15, R16, R17, R18, R19, R2, R20, R21, R22, R23, R24, R25, R26, R27, R28, R29, R30, R31, R32, R33, R34, R35, R36, R37, R38, R39, R4, R40, R41, R42, R43, R44, R45, R46, R47, R48, R49, R5, R50, R51, R52, R53, R54, R55, R56, R57, R58, R59, R60, R61, R62, R63, R64, R65, R66, R67, R68, R69, R7, R70, R8, R9, U76: moved to B.Cu
- C21: value 20pF -> 0.1uF
- C23, C25, C27, C29, C31, C33, C35, C37, C39, C41, C43, C45, C47, C49, C51, C53, C55, C57, C59, C61, C63, C65, C67, C69, C71, C73, C75, C77, C79, C81, C83: value 20pF -> 0.1uF; moved to B.Cu
- LED1: renamed from D1; value SK6812MINI -> SK6812MINI-E; footprint LED_SMD:LED_SK6812MINI_PLCC4_3.5x3.5mm_P1.75mm -> PCM_marbastlib-various:LED_6028R
- U10, U11, U12, U13, U14, U15, U16, U17, U18, U19, U20, U22, U23, U24, U25, U26, U27, U28, U29, U31, U32, U33, U34, U35, U36, U37, U38, U40, U41, U42, U43, U44, U45, U46, U47, U48, U49, U50, U51, U52, U53, U54, U55, U56, U57, U58, U59, U6, U60, U61, U62, U63, U64, U65, U66, U67, U68, U69, U7, U70, U71, U8, U9: value TMR2652D -> CT100LW-HD6; footprint prometheus-65-footprints:TMR2652D -> prometheus-65-footprints:CT100LW-HD6; moved to B.Cu
- U4: value TMR2652D -> CT100LW-HD6; footprint prometheus-65-footprints:TMR2652D -> prometheus-65-footprints:CT100LW-HD6
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Connections:
- C21 pad 2: Net-(U4-VREF) -> +3.3VA
- C23 pad 2: Net-(U6-VREF) -> +3.3VA
- C25 pad 2: Net-(U7-VREF) -> +3.3VA
- C27 pad 2: Net-(U8-VREF) -> +3.3VA
- C29 pad 2: Net-(U9-VREF) -> +3.3VA
- C31 pad 2: Net-(U10-VREF) -> +3.3VA
- C33 pad 2: Net-(U11-VREF) -> +3.3VA
- C35 pad 2: Net-(U12-VREF) -> +3.3VA
- C37 pad 2: Net-(U13-VREF) -> +3.3VA
- C39 pad 2: Net-(U14-VREF) -> +3.3VA
- C41 pad 2: Net-(U15-VREF) -> +3.3VA
- C43 pad 2: Net-(U16-VREF) -> +3.3VA
- C45 pad 2: Net-(U17-VREF) -> +3.3VA
- C47 pad 2: Net-(U18-VREF) -> +3.3VA
- C49 pad 2: Net-(U19-VREF) -> +3.3VA
- C51 pad 2: Net-(U20-VREF) -> +3.3VA
- C53 pad 2: Net-(U22-VREF) -> +3.3VA
- C55 pad 2: Net-(U23-VREF) -> +3.3VA
- C57 pad 2: Net-(U24-VREF) -> +3.3VA
- C59 pad 2: Net-(U25-VREF) -> +3.3VA
- C61 pad 2: Net-(U26-VREF) -> +3.3VA
- C63 pad 2: Net-(U27-VREF) -> +3.3VA
- C65 pad 2: Net-(U28-VREF) -> +3.3VA
- C67 pad 2: Net-(U29-VREF) -> +3.3VA
- C69 pad 2: Net-(U31-VREF) -> +3.3VA
- C71 pad 2: Net-(U32-VREF) -> +3.3VA
- C73 pad 2: Net-(U33-VREF) -> +3.3VA
- C75 pad 2: Net-(U34-VREF) -> +3.3VA
- C77 pad 2: Net-(U35-VREF) -> +3.3VA
- C79 pad 2: Net-(U36-VREF) -> +3.3VA
- C81 pad 2: Net-(U37-VREF) -> +3.3VA
- C83 pad 2: Net-(U38-VREF) -> +3.3VA
- LED1 pad 1: Net-(D1-DOUT) -> +5V
- LED1 pad 2: GND -> Net-(LED1-DOUT)
- LED1 pad 4: +5V -> GND
- R10 pad 1: Net-(U9-VOUT) -> Net-(U9-X1)
- R11 pad 1: Net-(U10-VOUT) -> Net-(U10-X1)
- R12 pad 1: Net-(U11-VOUT) -> Net-(U11-X1)
- R13 pad 1: Net-(U12-VOUT) -> Net-(U12-X1)
- R14 pad 1: Net-(U13-VOUT) -> Net-(U13-X1)
- R15 pad 1: Net-(U14-VOUT) -> Net-(U14-X1)
- R16 pad 1: Net-(U15-VOUT) -> Net-(U15-X1)
- R17 pad 1: Net-(U16-VOUT) -> Net-(U16-X1)
- R18 pad 1: Net-(U17-VOUT) -> Net-(U17-X1)
- R19 pad 1: Net-(U18-VOUT) -> Net-(U18-X1)
- R20 pad 1: Net-(U19-VOUT) -> Net-(U19-X1)
- R21 pad 1: Net-(U20-VOUT) -> Net-(U20-X1)
- R22 pad 1: Net-(U22-VOUT) -> Net-(U22-X1)
- R23 pad 1: Net-(U23-VOUT) -> Net-(U23-X1)
- R24 pad 1: Net-(U24-VOUT) -> Net-(U24-X1)
- R25 pad 1: Net-(U25-VOUT) -> Net-(U25-X1)
- R26 pad 1: Net-(U26-VOUT) -> Net-(U26-X1)
- R27 pad 1: Net-(U27-VOUT) -> Net-(U27-X1)
- R28 pad 1: Net-(U28-VOUT) -> Net-(U28-X1)
- R29 pad 1: Net-(U29-VOUT) -> Net-(U29-X1)
- R30 pad 1: Net-(U31-VOUT) -> Net-(U31-X1)
- R31 pad 1: Net-(U32-VOUT) -> Net-(U32-X1)
- R32 pad 1: Net-(U33-VOUT) -> Net-(U33-X1)
- R33 pad 1: Net-(U34-VOUT) -> Net-(U34-X1)
- R34 pad 1: Net-(U35-VOUT) -> Net-(U35-X1)
- R35 pad 1: Net-(U36-VOUT) -> Net-(U36-X1)
- R36 pad 1: Net-(U37-VOUT) -> Net-(U37-X1)
- R37 pad 1: Net-(U38-VOUT) -> Net-(U38-X1)
- R38 pad 1: Net-(U40-VOUT) -> Net-(U40-X1)
- R39 pad 1: Net-(U41-VOUT) -> Net-(U41-X1)
- R40 pad 1: Net-(U42-VOUT) -> Net-(U42-X1)
- R41 pad 1: Net-(U43-VOUT) -> Net-(U43-X1)
- R42 pad 1: Net-(U44-VOUT) -> Net-(U44-X1)
- R43 pad 1: Net-(U45-VOUT) -> Net-(U45-X1)
- R44 pad 1: Net-(U46-VOUT) -> Net-(U46-X1)
- R45 pad 1: Net-(U47-VOUT) -> Net-(U47-X1)
- R46 pad 1: Net-(U48-VOUT) -> Net-(U48-X1)
- R47 pad 1: Net-(U49-VOUT) -> Net-(U49-X1)
- R48 pad 1: Net-(U50-VOUT) -> Net-(U50-X1)
- R49 pad 1: Net-(U51-VOUT) -> Net-(U51-X1)
- R50 pad 1: Net-(U52-VOUT) -> Net-(U52-X1)
- R51 pad 1: Net-(U53-VOUT) -> Net-(U53-X1)
- R52 pad 1: Net-(U54-VOUT) -> Net-(U54-X1)
- R53 pad 1: Net-(U55-VOUT) -> Net-(U55-X1)
- R54 pad 1: Net-(U56-VOUT) -> Net-(U56-X1)
- R55 pad 1: Net-(U57-VOUT) -> Net-(U57-X1)
- R56 pad 1: Net-(U58-VOUT) -> Net-(U58-X1)
- R57 pad 1: Net-(U59-VOUT) -> Net-(U59-X1)
- R58 pad 1: Net-(U60-VOUT) -> Net-(U60-X1)
- R59 pad 1: Net-(U61-VOUT) -> Net-(U61-X1)
- R6 pad 1: Net-(U4-VOUT) -> Net-(U4-X1)
- R60 pad 1: Net-(U62-VOUT) -> Net-(U62-X1)
- R61 pad 1: Net-(U63-VOUT) -> Net-(U63-X1)
- R62 pad 1: Net-(U64-VOUT) -> Net-(U64-X1)
- R63 pad 1: Net-(U65-VOUT) -> Net-(U65-X1)
- R64 pad 1: Net-(U66-VOUT) -> Net-(U66-X1)
- R65 pad 1: Net-(U67-VOUT) -> Net-(U67-X1)
- R66 pad 1: Net-(U68-VOUT) -> Net-(U68-X1)
- R67 pad 1: Net-(U69-VOUT) -> Net-(U69-X1)
- R68 pad 1: Net-(U70-VOUT) -> Net-(U70-X1)
- R69 pad 1: Net-(U71-VOUT) -> Net-(U71-X1)
- R7 pad 1: Net-(U6-VOUT) -> Net-(U6-X1)
- R8 pad 1: Net-(U7-VOUT) -> Net-(U7-X1)
- R9 pad 1: Net-(U8-VOUT) -> Net-(U8-X1)
- U10 pad 1: Net-(U10-VREF) -> unconnected-(U10-X2-Pad1)
- U10 pad 2: GND -> unconnected-(U10-NC-Pad2)
- U10 pad 3: unconnected-(U10-Comp-Pad3) -> Net-(U10-X1)
- U10 pad 4: Net-(U10-VOUT) -> GND
- U10 pad 5: +3.3VA -> unconnected-(U10-NC-Pad5)
- U10 pad 6: unconnected-(U10-NC-Pad6) -> +3.3VA
- U10 pad 7: GND -> (no net)
- U11 pad 1: Net-(U11-VREF) -> unconnected-(U11-X2-Pad1)
- U11 pad 2: GND -> unconnected-(U11-NC-Pad2)
- U11 pad 3: unconnected-(U11-Comp-Pad3) -> Net-(U11-X1)
- U11 pad 4: Net-(U11-VOUT) -> GND
- U11 pad 5: +3.3VA -> unconnected-(U11-NC-Pad5)
- U11 pad 6: unconnected-(U11-NC-Pad6) -> +3.3VA
- U11 pad 7: GND -> (no net)
- U12 pad 1: Net-(U12-VREF) -> unconnected-(U12-X2-Pad1)
- U12 pad 2: GND -> unconnected-(U12-NC-Pad2)
- U12 pad 3: unconnected-(U12-Comp-Pad3) -> Net-(U12-X1)
- U12 pad 4: Net-(U12-VOUT) -> GND
- U12 pad 5: +3.3VA -> unconnected-(U12-NC-Pad5)
- U12 pad 6: unconnected-(U12-NC-Pad6) -> +3.3VA
- U12 pad 7: GND -> (no net)
- U13 pad 1: Net-(U13-VREF) -> unconnected-(U13-X2-Pad1)
- U13 pad 2: GND -> unconnected-(U13-NC-Pad2)
- U13 pad 3: unconnected-(U13-Comp-Pad3) -> Net-(U13-X1)
- U13 pad 4: Net-(U13-VOUT) -> GND
- U13 pad 5: +3.3VA -> unconnected-(U13-NC-Pad5)
- U13 pad 6: unconnected-(U13-NC-Pad6) -> +3.3VA
- U13 pad 7: GND -> (no net)
- U14 pad 1: Net-(U14-VREF) -> unconnected-(U14-X2-Pad1)
- U14 pad 2: GND -> unconnected-(U14-NC-Pad2)
- U14 pad 3: unconnected-(U14-Comp-Pad3) -> Net-(U14-X1)
- U14 pad 4: Net-(U14-VOUT) -> GND
- U14 pad 5: +3.3VA -> unconnected-(U14-NC-Pad5)
- U14 pad 6: unconnected-(U14-NC-Pad6) -> +3.3VA
- U14 pad 7: GND -> (no net)
- U15 pad 1: Net-(U15-VREF) -> unconnected-(U15-X2-Pad1)
- U15 pad 2: GND -> unconnected-(U15-NC-Pad2)
- U15 pad 3: unconnected-(U15-Comp-Pad3) -> Net-(U15-X1)
- U15 pad 4: Net-(U15-VOUT) -> GND
- U15 pad 5: +3.3VA -> unconnected-(U15-NC-Pad5)
- U15 pad 6: unconnected-(U15-NC-Pad6) -> +3.3VA
- U15 pad 7: GND -> (no net)
- U16 pad 1: Net-(U16-VREF) -> unconnected-(U16-X2-Pad1)
- U16 pad 2: GND -> unconnected-(U16-NC-Pad2)
- U16 pad 3: unconnected-(U16-Comp-Pad3) -> Net-(U16-X1)
- U16 pad 4: Net-(U16-VOUT) -> GND
- U16 pad 5: +3.3VA -> unconnected-(U16-NC-Pad5)
- U16 pad 6: unconnected-(U16-NC-Pad6) -> +3.3VA
- U16 pad 7: GND -> (no net)
- U17 pad 1: Net-(U17-VREF) -> unconnected-(U17-X2-Pad1)
- U17 pad 2: GND -> unconnected-(U17-NC-Pad2)
- U17 pad 3: unconnected-(U17-Comp-Pad3) -> Net-(U17-X1)
- U17 pad 4: Net-(U17-VOUT) -> GND
- U17 pad 5: +3.3VA -> unconnected-(U17-NC-Pad5)
- U17 pad 6: unconnected-(U17-NC-Pad6) -> +3.3VA
- U17 pad 7: GND -> (no net)
- U18 pad 1: Net-(U18-VREF) -> unconnected-(U18-X2-Pad1)
- U18 pad 2: GND -> unconnected-(U18-NC-Pad2)
- U18 pad 3: unconnected-(U18-Comp-Pad3) -> Net-(U18-X1)
- U18 pad 4: Net-(U18-VOUT) -> GND
- U18 pad 5: +3.3VA -> unconnected-(U18-NC-Pad5)
- U18 pad 6: unconnected-(U18-NC-Pad6) -> +3.3VA
- U18 pad 7: GND -> (no net)
- U19 pad 1: Net-(U19-VREF) -> unconnected-(U19-X2-Pad1)
- U19 pad 2: GND -> unconnected-(U19-NC-Pad2)
- U19 pad 3: unconnected-(U19-Comp-Pad3) -> Net-(U19-X1)
- U19 pad 4: Net-(U19-VOUT) -> GND
- U19 pad 5: +3.3VA -> unconnected-(U19-NC-Pad5)
- U19 pad 6: unconnected-(U19-NC-Pad6) -> +3.3VA
- U19 pad 7: GND -> (no net)
- U20 pad 1: Net-(U20-VREF) -> unconnected-(U20-X2-Pad1)
- U20 pad 2: GND -> unconnected-(U20-NC-Pad2)
- U20 pad 3: unconnected-(U20-Comp-Pad3) -> Net-(U20-X1)
- U20 pad 4: Net-(U20-VOUT) -> GND
- U20 pad 5: +3.3VA -> unconnected-(U20-NC-Pad5)
- U20 pad 6: unconnected-(U20-NC-Pad6) -> +3.3VA
- U20 pad 7: GND -> (no net)
- U22 pad 1: Net-(U22-VREF) -> unconnected-(U22-X2-Pad1)
- U22 pad 2: GND -> unconnected-(U22-NC-Pad2)
- U22 pad 3: unconnected-(U22-Comp-Pad3) -> Net-(U22-X1)
- U22 pad 4: Net-(U22-VOUT) -> GND
- U22 pad 5: +3.3VA -> unconnected-(U22-NC-Pad5)
- U22 pad 6: unconnected-(U22-NC-Pad6) -> +3.3VA
- U22 pad 7: GND -> (no net)
- U23 pad 1: Net-(U23-VREF) -> unconnected-(U23-X2-Pad1)
- U23 pad 2: GND -> unconnected-(U23-NC-Pad2)
- U23 pad 3: unconnected-(U23-Comp-Pad3) -> Net-(U23-X1)
- U23 pad 4: Net-(U23-VOUT) -> GND
- U23 pad 5: +3.3VA -> unconnected-(U23-NC-Pad5)
- U23 pad 6: unconnected-(U23-NC-Pad6) -> +3.3VA
- U23 pad 7: GND -> (no net)
- U24 pad 1: Net-(U24-VREF) -> unconnected-(U24-X2-Pad1)
- U24 pad 2: GND -> unconnected-(U24-NC-Pad2)
- U24 pad 3: unconnected-(U24-Comp-Pad3) -> Net-(U24-X1)
- U24 pad 4: Net-(U24-VOUT) -> GND
- U24 pad 5: +3.3VA -> unconnected-(U24-NC-Pad5)
- U24 pad 6: unconnected-(U24-NC-Pad6) -> +3.3VA
- U24 pad 7: GND -> (no net)
- U25 pad 1: Net-(U25-VREF) -> unconnected-(U25-X2-Pad1)
- U25 pad 2: GND -> unconnected-(U25-NC-Pad2)
- U25 pad 3: unconnected-(U25-Comp-Pad3) -> Net-(U25-X1)
- U25 pad 4: Net-(U25-VOUT) -> GND
- U25 pad 5: +3.3VA -> unconnected-(U25-NC-Pad5)
- U25 pad 6: unconnected-(U25-NC-Pad6) -> +3.3VA
- U25 pad 7: GND -> (no net)
- U26 pad 1: Net-(U26-VREF) -> unconnected-(U26-X2-Pad1)
- U26 pad 2: GND -> unconnected-(U26-NC-Pad2)
- U26 pad 3: unconnected-(U26-Comp-Pad3) -> Net-(U26-X1)
- U26 pad 4: Net-(U26-VOUT) -> GND
- U26 pad 5: +3.3VA -> unconnected-(U26-NC-Pad5)
- U26 pad 6: unconnected-(U26-NC-Pad6) -> +3.3VA
- U26 pad 7: GND -> (no net)
- U27 pad 1: Net-(U27-VREF) -> unconnected-(U27-X2-Pad1)
- U27 pad 2: GND -> unconnected-(U27-NC-Pad2)
- U27 pad 3: unconnected-(U27-Comp-Pad3) -> Net-(U27-X1)
- U27 pad 4: Net-(U27-VOUT) -> GND
- U27 pad 5: +3.3VA -> unconnected-(U27-NC-Pad5)
- U27 pad 6: unconnected-(U27-NC-Pad6) -> +3.3VA
- U27 pad 7: GND -> (no net)
- U28 pad 1: Net-(U28-VREF) -> unconnected-(U28-X2-Pad1)
- U28 pad 2: GND -> unconnected-(U28-NC-Pad2)
- U28 pad 3: unconnected-(U28-Comp-Pad3) -> Net-(U28-X1)
- U28 pad 4: Net-(U28-VOUT) -> GND
- U28 pad 5: +3.3VA -> unconnected-(U28-NC-Pad5)
- U28 pad 6: unconnected-(U28-NC-Pad6) -> +3.3VA
- U28 pad 7: GND -> (no net)
- U29 pad 1: Net-(U29-VREF) -> unconnected-(U29-X2-Pad1)
- U29 pad 2: GND -> unconnected-(U29-NC-Pad2)
- U29 pad 3: unconnected-(U29-Comp-Pad3) -> Net-(U29-X1)
- U29 pad 4: Net-(U29-VOUT) -> GND
- U29 pad 5: +3.3VA -> unconnected-(U29-NC-Pad5)
- U29 pad 6: unconnected-(U29-NC-Pad6) -> +3.3VA
- U29 pad 7: GND -> (no net)
- U31 pad 1: Net-(U31-VREF) -> unconnected-(U31-X2-Pad1)
- U31 pad 2: GND -> unconnected-(U31-NC-Pad2)
- U31 pad 3: unconnected-(U31-Comp-Pad3) -> Net-(U31-X1)
- U31 pad 4: Net-(U31-VOUT) -> GND
- U31 pad 5: +3.3VA -> unconnected-(U31-NC-Pad5)
- U31 pad 6: unconnected-(U31-NC-Pad6) -> +3.3VA
- U31 pad 7: GND -> (no net)
- U32 pad 1: Net-(U32-VREF) -> unconnected-(U32-X2-Pad1)
- U32 pad 2: GND -> unconnected-(U32-NC-Pad2)
- U32 pad 3: unconnected-(U32-Comp-Pad3) -> Net-(U32-X1)
- U32 pad 4: Net-(U32-VOUT) -> GND
- U32 pad 5: +3.3VA -> unconnected-(U32-NC-Pad5)
- U32 pad 6: unconnected-(U32-NC-Pad6) -> +3.3VA
- U32 pad 7: GND -> (no net)
- U33 pad 1: Net-(U33-VREF) -> unconnected-(U33-X2-Pad1)
- U33 pad 2: GND -> unconnected-(U33-NC-Pad2)
- U33 pad 3: unconnected-(U33-Comp-Pad3) -> Net-(U33-X1)
- U33 pad 4: Net-(U33-VOUT) -> GND
- U33 pad 5: +3.3VA -> unconnected-(U33-NC-Pad5)
- U33 pad 6: unconnected-(U33-NC-Pad6) -> +3.3VA
- U33 pad 7: GND -> (no net)
- U34 pad 1: Net-(U34-VREF) -> unconnected-(U34-X2-Pad1)
- U34 pad 2: GND -> unconnected-(U34-NC-Pad2)
- U34 pad 3: unconnected-(U34-Comp-Pad3) -> Net-(U34-X1)
- U34 pad 4: Net-(U34-VOUT) -> GND
- U34 pad 5: +3.3VA -> unconnected-(U34-NC-Pad5)
- U34 pad 6: unconnected-(U34-NC-Pad6) -> +3.3VA
- U34 pad 7: GND -> (no net)
- U35 pad 1: Net-(U35-VREF) -> unconnected-(U35-X2-Pad1)
- U35 pad 2: GND -> unconnected-(U35-NC-Pad2)
- U35 pad 3: unconnected-(U35-Comp-Pad3) -> Net-(U35-X1)
- U35 pad 4: Net-(U35-VOUT) -> GND
- U35 pad 5: +3.3VA -> unconnected-(U35-NC-Pad5)
- U35 pad 6: unconnected-(U35-NC-Pad6) -> +3.3VA
- U35 pad 7: GND -> (no net)
- U36 pad 1: Net-(U36-VREF) -> unconnected-(U36-X2-Pad1)
- U36 pad 2: GND -> unconnected-(U36-NC-Pad2)
- U36 pad 3: unconnected-(U36-Comp-Pad3) -> Net-(U36-X1)
- U36 pad 4: Net-(U36-VOUT) -> GND
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Routing:
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Other:
- board outline added: 3.6 x 3.3 mm

Commit message: feat: working changes
Parts:
- removed C23, C24, C25, C26, C27, C28, C29, C30, C31, C32, C33, C34, C35, C36, C37, C38, C39, C40, C41, C42, C43, C44, C45, C46, C47, C48, C49, C50, C51, C52, C53, C54, C55, C56, C57, C58, C59, C60, C61, C62, C63, C64, C65, C66, C67, C68, C69, C70, C71, C72, C73, C74, C75, C76, C77, C78, C79, C80, C81, C82, C83: 0.1uF, Capacitor_SMD:C_0402_1005Metric
- removed R10, R11, R12, R13, R14, R16, R17, R18, R19, R20, R21, R22, R23, R24, R25, R26, R27, R28, R29, R30, R31, R32, R33, R36, R37, R38, R39, R40, R41, R42, R43, R44, R45, R46, R47, R48, R49, R50, R51, R52, R53, R54, R55, R56, R57, R58, R59, R6, R60, R61, R62, R63, R64, R65, R66, R67, R68, R69, R7, R8, R9: 1kΩ, Resistor_SMD:R_0402_1005Metric
- removed R3: 1MΩ, Resistor_SMD:R_0603_1608Metric
- removed R4, R5: 22Ω, Resistor_SMD:R_0603_1608Metric
- removed R70: 330Ω, Resistor_SMD:R_0603_1608Metric
- removed U1: STM32F405RGTx, Package_QFP:LQFP-64_10x10mm_P0.5mm
- removed U2: TPS7A4700, prometheus-65-footprints:TPS7A47000RGWT
- added LED65: SK6812MINI-E, PCM_marbastlib-various:LED_6028R, B.Cu at (157.2, 109.2)
- added LED66: SK6812MINI-E, PCM_marbastlib-various:LED_6028R, B.Cu at (176.2, 109.2)
- added LED67: SK6812MINI-E, PCM_marbastlib-various:LED_6028R, B.Cu at (195.3, 109.2)
- added LED68: SK6812MINI-E, PCM_marbastlib-various:LED_6028R, B.Cu at (214.3, 109.2)
- added LED69: SK6812MINI-E, PCM_marbastlib-various:LED_6028R, B.Cu at (233.4, 109.2)
- added LED70: SK6812MINI-E, PCM_marbastlib-various:LED_6028R, B.Cu at (252.4, 109.2)
- added LED71: SK6812MINI-E, PCM_marbastlib-various:LED_6028R, B.Cu at (278.6, 109.2)
- added LED72: SK6812MINI-E, PCM_marbastlib-various:LED_6028R, B.Cu at (304.8, 109.2)
- added LED73: SK6812MINI-E, PCM_marbastlib-various:LED_6028R, B.Cu at (323.9, 109.2)
- added LED74: SK6812MINI-E, PCM_marbastlib-various:LED_6028R, B.Cu at (40.5, 128.3)
- added LED75: SK6812MINI-E, PCM_marbastlib-various:LED_6028R, B.Cu at (64.3, 128.3)
- added LED76: SK6812MINI-E, PCM_marbastlib-various:LED_6028R, B.Cu at (88.1, 128.3)
- added LED77: SK6812MINI-E, PCM_marbastlib-various:LED_6028R, B.Cu at (159.5, 128.3)
- added LED78: SK6812MINI-E, PCM_marbastlib-various:LED_6028R, B.Cu at (228.6, 128.3)
- added LED79: SK6812MINI-E, PCM_marbastlib-various:LED_6028R, B.Cu at (247.7, 128.3)
- added LED80: SK6812MINI-E, PCM_marbastlib-various:LED_6028R, B.Cu at (266.7, 128.3)
- added LED81: SK6812MINI-E, PCM_marbastlib-various:LED_6028R, B.Cu at (285.8, 128.3)
- added LED82: SK6812MINI-E, PCM_marbastlib-various:LED_6028R, B.Cu at (304.8, 128.3)
- added LED83: SK6812MINI-E, PCM_marbastlib-various:LED_6028R, B.Cu at (323.9, 128.3)
- added LED84: SK6812MINI-E, PCM_marbastlib-various:LED_6028R, B.Cu at (207.0, -93.5)
- added S65: 1.00u, ScottoKeebs_Hotswap:Hotswap_MX_Plated_1.00u, F.Cu at (157.2, 114.3)
- added S66: 1.00u, ScottoKeebs_Hotswap:Hotswap_MX_Plated_1.00u, F.Cu at (176.2, 114.3)
- added S67: 1.00u, ScottoKeebs_Hotswap:Hotswap_MX_Plated_1.00u, F.Cu at (195.3, 114.3)
- added S68: 1.00u, ScottoKeebs_Hotswap:Hotswap_MX_Plated_1.00u, F.Cu at (214.3, 114.3)
- added S69: 1.00u, ScottoKeebs_Hotswap:Hotswap_MX_Plated_1.00u, F.Cu at (233.4, 114.3)
- added S70: 1.00u, ScottoKeebs_Hotswap:Hotswap_MX_Plated_1.00u, F.Cu at (252.4, 114.3)
- added S71: 1.00u, ScottoKeebs_Hotswap:Hotswap_MX_Plated_1.00u, F.Cu at (278.6, 114.3)
- added S72: 1.00u, ScottoKeebs_Hotswap:Hotswap_MX_Plated_1.00u, F.Cu at (304.8, 114.3)
- added S73: 1.00u, ScottoKeebs_Hotswap:Hotswap_MX_Plated_1.00u, F.Cu at (323.9, 114.3)
- added S74: 1.00u, ScottoKeebs_Hotswap:Hotswap_MX_Plated_1.00u, F.Cu at (40.5, 133.3)
- added S75: 1.00u, ScottoKeebs_Hotswap:Hotswap_MX_Plated_1.00u, F.Cu at (64.3, 133.3)
- added S76: 1.00u, ScottoKeebs_Hotswap:Hotswap_MX_Plated_1.00u, F.Cu at (88.1, 133.3)
- added S77: 1.00u, ScottoKeebs_Hotswap:Hotswap_MX_Plated_1.00u, F.Cu at (159.5, 133.3)
- added S78: 1.00u, ScottoKeebs_Hotswap:Hotswap_MX_Plated_1.00u, F.Cu at (228.6, 133.3)
- added S79: 1.00u, ScottoKeebs_Hotswap:Hotswap_MX_Plated_1.00u, F.Cu at (247.7, 133.3)
- added S80: 1.00u, ScottoKeebs_Hotswap:Hotswap_MX_Plated_1.00u, F.Cu at (266.7, 133.3)
- added S81: 1.00u, ScottoKeebs_Hotswap:Hotswap_MX_Plated_1.00u, F.Cu at (285.8, 133.3)
- added S82: 1.00u, ScottoKeebs_Hotswap:Hotswap_MX_Plated_1.00u, F.Cu at (304.8, 133.3)
- added S83: 1.00u, ScottoKeebs_Hotswap:Hotswap_MX_Plated_1.00u, F.Cu at (323.9, 133.3)
- added S84: 1.00u, ScottoKeebs_Hotswap:Hotswap_MX_Plated_1.00u, F.Cu at (207.0, -98.5)
- added SC1: 100nF, Capacitor_SMD:C_0402_1005Metric, B.Cu at (42.8, 33.8)
- added SC10: 100nF, Capacitor_SMD:C_0402_1005Metric, B.Cu at (214.3, 33.8)
- added SC11: 100nF, Capacitor_SMD:C_0402_1005Metric, B.Cu at (233.3, 33.8)
- added SC12: 100nF, Capacitor_SMD:C_0402_1005Metric, B.Cu at (252.4, 33.8)
- added SC13: 100nF, Capacitor_SMD:C_0402_1005Metric, B.Cu at (271.4, 33.8)
- added SC14: 100nF, Capacitor_SMD:C_0402_1005Metric, B.Cu at (290.5, 33.8)
- added SC15: 100nF, Capacitor_SMD:C_0402_1005Metric, B.Cu at (309.5, 33.8)
- added SC16: 100nF, Capacitor_SMD:C_0402_1005Metric, B.Cu at (42.8, 52.8)
- added SC17: 100nF, Capacitor_SMD:C_0402_1005Metric, B.Cu at (61.9, 52.8)
- added SC18: 100nF, Capacitor_SMD:C_0402_1005Metric, B.Cu at (80.9, 52.8)
- added SC19: 100nF, Capacitor_SMD:C_0402_1005Metric, B.Cu at (100.0, 52.8)
- added SC2: 100nF, Capacitor_SMD:C_0402_1005Metric, B.Cu at (61.9, 33.8)
- added SC20: 100nF, Capacitor_SMD:C_0402_1005Metric, B.Cu at (119.0, 52.8)
- added SC21: 100nF, Capacitor_SMD:C_0402_1005Metric, B.Cu at (138.1, 52.8)
- added SC22: 100nF, Capacitor_SMD:C_0402_1005Metric, B.Cu at (157.1, 52.8)
- added SC23: 100nF, Capacitor_SMD:C_0402_1005Metric, B.Cu at (176.2, 52.8)
- added SC24: 100nF, Capacitor_SMD:C_0402_1005Metric, B.Cu at (195.2, 52.8)
- added SC25: 100nF, Capacitor_SMD:C_0402_1005Metric, B.Cu at (214.3, 52.8)
- added SC26: 100nF, Capacitor_SMD:C_0402_1005Metric, B.Cu at (233.3, 52.8)
- added SC27: 100nF, Capacitor_SMD:C_0402_1005Metric, B.Cu at (252.4, 52.8)
- added SC28: 100nF, Capacitor_SMD:C_0402_1005Metric, B.Cu at (271.4, 52.8)
- added SC29: 100nF, Capacitor_SMD:C_0402_1005Metric, B.Cu at (300.0, 52.8)
- added SC3: 100nF, Capacitor_SMD:C_0402_1005Metric, B.Cu at (80.9, 33.8)
- added SC30: 100nF, Capacitor_SMD:C_0402_1005Metric, B.Cu at (328.6, 52.8)
- added SC31: 100nF, Capacitor_SMD:C_0402_1005Metric, B.Cu at (47.6, 71.9)
- added SC32: 100nF, Capacitor_SMD:C_0402_1005Metric, B.Cu at (71.4, 71.9)
- added SC33: 100nF, Capacitor_SMD:C_0402_1005Metric, B.Cu at (90.5, 71.9)
- added SC34: 100nF, Capacitor_SMD:C_0402_1005Metric, B.Cu at (109.5, 71.9)
- added SC35: 100nF, Capacitor_SMD:C_0402_1005Metric, B.Cu at (128.6, 71.9)
- added SC36: 100nF, Capacitor_SMD:C_0402_1005Metric, B.Cu at (147.6, 71.9)
- added SC37: 100nF, Capacitor_SMD:C_0402_1005Metric, B.Cu at (166.7, 71.9)
- added SC38: 100nF, Capacitor_SMD:C_0402_1005Metric, B.Cu at (185.7, 71.9)
- added SC39: 100nF, Capacitor_SMD:C_0402_1005Metric, B.Cu at (204.8, 71.9)
- added SC4: 100nF, Capacitor_SMD:C_0402_1005Metric, B.Cu at (100.0, 33.8)
- added SC40: 100nF, Capacitor_SMD:C_0402_1005Metric, B.Cu at (223.8, 71.9)
- added SC41: 100nF, Capacitor_SMD:C_0402_1005Metric, B.Cu at (242.8, 71.9)
- added SC42: 100nF, Capacitor_SMD:C_0402_1005Metric, B.Cu at (261.9, 71.9)
- added SC43: 100nF, Capacitor_SMD:C_0402_1005Metric, B.Cu at (280.9, 71.9)
- added SC44: 100nF, Capacitor_SMD:C_0402_1005Metric, B.Cu at (304.8, 71.9)
- added SC45: 100nF, Capacitor_SMD:C_0402_1005Metric, B.Cu at (328.6, 71.9)
- added SC46: 100nF, Capacitor_SMD:C_0402_1005Metric, B.Cu at (50.0, 90.9)
- added SC47: 100nF, Capacitor_SMD:C_0402_1005Metric, B.Cu at (76.2, 90.9)
- added SC48: 100nF, Capacitor_SMD:C_0402_1005Metric, B.Cu at (95.2, 90.9)
- added SC49: 100nF, Capacitor_SMD:C_0402_1005Metric, B.Cu at (114.3, 90.9)
- added SC5: 100nF, Capacitor_SMD:C_0402_1005Metric, B.Cu at (119.0, 33.8)
- added SC50: 100nF, Capacitor_SMD:C_0402_1005Metric, B.Cu at (133.3, 90.9)
- added SC51: 100nF, Capacitor_SMD:C_0402_1005Metric, B.Cu at (152.4, 90.9)
- added SC52: 100nF, Capacitor_SMD:C_0402_1005Metric, B.Cu at (171.4, 90.9)
- added SC53: 100nF, Capacitor_SMD:C_0402_1005Metric, B.Cu at (190.5, 90.9)
- added SC54: 100nF, Capacitor_SMD:C_0402_1005Metric, B.Cu at (209.5, 90.9)
- added SC55: 100nF, Capacitor_SMD:C_0402_1005Metric, B.Cu at (228.6, 90.9)
- added SC56: 100nF, Capacitor_SMD:C_0402_1005Metric, B.Cu at (247.6, 90.9)
- added SC57: 100nF, Capacitor_SMD:C_0402_1005Metric, B.Cu at (266.7, 90.9)
- added SC58: 100nF, Capacitor_SMD:C_0402_1005Metric, B.Cu at (297.6, 90.9)
- added SC59: 100nF, Capacitor_SMD:C_0402_1005Metric, B.Cu at (328.6, 90.9)
- added SC6: 100nF, Capacitor_SMD:C_0402_1005Metric, B.Cu at (138.1, 33.8)
- added SC60: 100nF, Capacitor_SMD:C_0402_1005Metric, B.Cu at (54.7, 110.0)
- added SC61: 100nF, Capacitor_SMD:C_0402_1005Metric, B.Cu at (85.7, 110.0)
- added SC62: 100nF, Capacitor_SMD:C_0402_1005Metric, B.Cu at (104.7, 110.0)
- added SC63: 100nF, Capacitor_SMD:C_0402_1005Metric, B.Cu at (123.8, 110.0)
- added SC64: 100nF, Capacitor_SMD:C_0402_1005Metric, B.Cu at (142.8, 110.0)
- added SC65: 100nF, Capacitor_SMD:C_0402_1005Metric, B.Cu at (161.9, 110.0)
- added SC66: 100nF, Capacitor_SMD:C_0402_1005Metric, B.Cu at (180.9, 110.0)
- added SC67: 100nF, Capacitor_SMD:C_0402_1005Metric, B.Cu at (200.0, 110.0)
- added SC68: 100nF, Capacitor_SMD:C_0402_1005Metric, B.Cu at (219.0, 110.0)
- added SC69: 100nF, Capacitor_SMD:C_0402_1005Metric, B.Cu at (238.1, 110.0)
- added SC7: 100nF, Capacitor_SMD:C_0402_1005Metric, B.Cu at (157.1, 33.8)
- added SC70: 100nF, Capacitor_SMD:C_0402_1005Metric, B.Cu at (257.1, 110.0)
- added SC71: 100nF, Capacitor_SMD:C_0402_1005Metric, B.Cu at (283.3, 110.0)
- added SC72: 100nF, Capacitor_SMD:C_0402_1005Metric, B.Cu at (309.5, 110.0)
- added SC73: 100nF, Capacitor_SMD:C_0402_1005Metric, B.Cu at (328.6, 110.0)
- added SC74: 100nF, Capacitor_SMD:C_0402_1005Metric, B.Cu at (45.2, 129.0)
- added SC75: 100nF, Capacitor_SMD:C_0402_1005Metric, B.Cu at (69.0, 129.0)
- added SC76: 100nF, Capacitor_SMD:C_0402_1005Metric, B.Cu at (92.8, 129.0)
- added SC77: 100nF, Capacitor_SMD:C_0402_1005Metric, B.Cu at (164.3, 129.0)
- added SC78: 100nF, Capacitor_SMD:C_0402_1005Metric, B.Cu at (233.3, 129.0)
- added SC79: 100nF, Capacitor_SMD:C_0402_1005Metric, B.Cu at (252.4, 129.0)
- added SC8: 100nF, Capacitor_SMD:C_0402_1005Metric, B.Cu at (176.2, 33.8)
- added SC80: 100nF, Capacitor_SMD:C_0402_1005Metric, B.Cu at (271.4, 129.0)
- added SC81: 100nF, Capacitor_SMD:C_0402_1005Metric, B.Cu at (290.5, 129.0)
- added SC82: 100nF, Capacitor_SMD:C_0402_1005Metric, B.Cu at (309.5, 129.0)
- added SC83: 100nF, Capacitor_SMD:C_0402_1005Metric, B.Cu at (328.6, 129.0)
- added SC84: 100nF, Capacitor_SMD:C_0402_1005Metric, B.Cu at (202.2, -94.2)
- added SC9: 100nF, Capacitor_SMD:C_0402_1005Metric, B.Cu at (195.2, 33.8)
- added U100: ALT025-14E, prometheus-65-footprints:ALT025-14E, B.Cu at (39.8, 76.1)
- added U101: ALT025-14E, prometheus-65-footprints:ALT025-14E, B.Cu at (63.6, 76.1)
- added U102: ALT025-14E, prometheus-65-footprints:ALT025-14E, B.Cu at (82.6, 76.1)
- added U103: ALT025-14E, prometheus-65-footprints:ALT025-14E, B.Cu at (101.7, 76.1)
- added U104: ALT025-14E, prometheus-65-footprints:ALT025-14E, B.Cu at (120.7, 76.1)
- added U105: ALT025-14E, prometheus-65-footprints:ALT025-14E, B.Cu at (139.8, 76.1)
- added U106: ALT025-14E, prometheus-65-footprints:ALT025-14E, B.Cu at (158.8, 76.1)
- added U107: ALT025-14E, prometheus-65-footprints:ALT025-14E, B.Cu at (177.9, 76.1)
- added U108: ALT025-14E, prometheus-65-footprints:ALT025-14E, B.Cu at (196.9, 76.1)
- added U109: ALT025-14E, prometheus-65-footprints:ALT025-14E, B.Cu at (216.0, 76.1)
- added U110: ALT025-14E, prometheus-65-footprints:ALT025-14E, B.Cu at (235.0, 76.1)
- added U111: ALT025-14E, prometheus-65-footprints:ALT025-14E, B.Cu at (254.1, 76.1)
- added U112: ALT025-14E, prometheus-65-footprints:ALT025-14E, B.Cu at (273.1, 76.1)
- added U113: ALT025-14E, prometheus-65-footprints:ALT025-14E, B.Cu at (296.9, 76.1)
- added U114: ALT025-14E, prometheus-65-footprints:ALT025-14E, B.Cu at (320.7, 76.1)
- added U115: ALT025-14E, prometheus-65-footprints:ALT025-14E, B.Cu at (42.1, 95.2)
- added U116: ALT025-14E, prometheus-65-footprints:ALT025-14E, B.Cu at (68.3, 95.2)
- added U117: ALT025-14E, prometheus-65-footprints:ALT025-14E, B.Cu at (87.4, 95.2)
- added U118: ALT025-14E, prometheus-65-footprints:ALT025-14E, B.Cu at (106.4, 95.2)
- added U119: ALT025-14E, prometheus-65-footprints:ALT025-14E, B.Cu at (125.5, 95.2)
- added U120: ALT025-14E, prometheus-65-footprints:ALT025-14E, B.Cu at (144.5, 95.2)
- added U121: ALT025-14E, prometheus-65-footprints:ALT025-14E, B.Cu at (163.6, 95.2)
- added U122: ALT025-14E, prometheus-65-footprints:ALT025-14E, B.Cu at (182.6, 95.2)
- added U123: ALT025-14E, prometheus-65-footprints:ALT025-14E, B.Cu at (201.7, 95.2)
- added U124: ALT025-14E, prometheus-65-footprints:ALT025-14E, B.Cu at (220.7, 95.2)
- added U125: ALT025-14E, prometheus-65-footprints:ALT025-14E, B.Cu at (239.8, 95.2)
- added U126: ALT025-14E, prometheus-65-footprints:ALT025-14E, B.Cu at (258.8, 95.2)
- added U127: ALT025-14E, prometheus-65-footprints:ALT025-14E, B.Cu at (289.8, 95.2)
- added U128: ALT025-14E, prometheus-65-footprints:ALT025-14E, B.Cu at (320.7, 95.2)
- added U129: ALT025-14E, prometheus-65-footprints:ALT025-14E, B.Cu at (46.9, 114.2)
- added U130: ALT025-14E, prometheus-65-footprints:ALT025-14E, B.Cu at (77.8, 114.2)
- added U131: ALT025-14E, prometheus-65-footprints:ALT025-14E, B.Cu at (96.9, 114.2)
- added U132: ALT025-14E, prometheus-65-footprints:ALT025-14E, B.Cu at (116.0, 114.2)
- added U133: ALT025-14E, prometheus-65-footprints:ALT025-14E, B.Cu at (135.0, 114.2)
- added U134: ALT025-14E, prometheus-65-footprints:ALT025-14E, B.Cu at (154.1, 114.2)
- added U135: ALT025-14E, prometheus-65-footprints:ALT025-14E, B.Cu at (173.1, 114.2)
- added U136: ALT025-14E, prometheus-65-footprints:ALT025-14E, B.Cu at (192.2, 114.2)
- added U137: ALT025-14E, prometheus-65-footprints:ALT025-14E, B.Cu at (211.2, 114.2)
- added U138: ALT025-14E, prometheus-65-footprints:ALT025-14E, B.Cu at (230.2, 114.2)
- added U139: ALT025-14E, prometheus-65-footprints:ALT025-14E, B.Cu at (249.3, 114.2)
- added U140: ALT025-14E, prometheus-65-footprints:ALT025-14E, B.Cu at (275.5, 114.2)
- added U141: ALT025-14E, prometheus-65-footprints:ALT025-14E, B.Cu at (301.7, 114.2)
- added U142: ALT025-14E, prometheus-65-footprints:ALT025-14E, B.Cu at (320.7, 114.2)
- added U143: ALT025-14E, prometheus-65-footprints:ALT025-14E, B.Cu at (37.4, 133.2)
- added U144: ALT025-14E, prometheus-65-footprints:ALT025-14E, B.Cu at (61.2, 133.2)
- added U145: ALT025-14E, prometheus-65-footprints:ALT025-14E, B.Cu at (85.0, 133.2)
- added U146: ALT025-14E, prometheus-65-footprints:ALT025-14E, B.Cu at (156.4, 133.2)
- added U147: ALT025-14E, prometheus-65-footprints:ALT025-14E, B.Cu at (225.5, 133.2)
- added U148: ALT025-14E, prometheus-65-footprints:ALT025-14E, B.Cu at (244.5, 133.2)
- added U149: ALT025-14E, prometheus-65-footprints:ALT025-14E, B.Cu at (263.6, 133.2)
- added U150: ALT025-14E, prometheus-65-footprints:ALT025-14E, B.Cu at (282.6, 133.2)
- added U151: ALT025-14E, prometheus-65-footprints:ALT025-14E, B.Cu at (301.7, 133.2)
- added U152: ALT025-14E, prometheus-65-footprints:ALT025-14E, B.Cu at (320.7, 133.2)
- added U153: ALT025-14E, prometheus-65-footprints:ALT025-14E, B.Cu at (210.1, -98.5)
- added U21: TPD4E05U06DQAR, prometheus-65-footprints:TPD4E05U06DQAR, F.Cu at (280.0, -22.6)
- added U30: TPD4E05U06DQAR, prometheus-65-footprints:TPD4E05U06DQAR, F.Cu at (289.0, -34.7)
- added U39: TPD4E05U06DQAR, prometheus-65-footprints:TPD4E05U06DQAR, F.Cu at (297.9, -40.7)
- added U5: TPS7A4700, prometheus-65-footprints:TPS7A47000RGWT, F.Cu at (278.6, -57.5)
- added U72: ALT025-14E, prometheus-65-footprints:ALT025-14E, B.Cu at (73.1, 38.0)
- added U73: ALT025-14E, prometheus-65-footprints:ALT025-14E, B.Cu at (92.1, 38.0)
- added U74: ALT025-14E, prometheus-65-footprints:ALT025-14E, B.Cu at (111.2, 38.0)
- added U75: ALT025-14E, prometheus-65-footprints:ALT025-14E, B.Cu at (130.2, 38.0)
- added U77: ALT025-14E, prometheus-65-footprints:ALT025-14E, B.Cu at (168.3, 38.0)
- added U78: ALT025-14E, prometheus-65-footprints:ALT025-14E, B.Cu at (187.4, 38.0)
- added U79: ALT025-14E, prometheus-65-footprints:ALT025-14E, B.Cu at (206.4, 38.0)
- added U80: ALT025-14E, prometheus-65-footprints:ALT025-14E, B.Cu at (225.5, 38.0)
- added U81: ALT025-14E, prometheus-65-footprints:ALT025-14E, B.Cu at (244.5, 38.0)
- added U82: ALT025-14E, prometheus-65-footprints:ALT025-14E, B.Cu at (263.6, 38.0)
- added U83: ALT025-14E, prometheus-65-footprints:ALT025-14E, B.Cu at (282.6, 38.0)
- added U84: ALT025-14E, prometheus-65-footprints:ALT025-14E, B.Cu at (301.7, 38.0)
- added U85: ALT025-14E, prometheus-65-footprints:ALT025-14E, B.Cu at (35.0, 57.0)
- added U86: ALT025-14E, prometheus-65-footprints:ALT025-14E, B.Cu at (54.0, 57.0)
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Connections:
- net Net-(LED1-DOUT) renamed /Key_1/DOUT
- net Net-(LED10-DIN) renamed /Key_10/DIN
- net Net-(LED10-DOUT) renamed /Key_10/DOUT
- net Net-(LED11-DOUT) renamed /Key_11/DOUT
- net Net-(LED12-DOUT) renamed /Key_12/DOUT
- net Net-(LED13-DOUT) renamed /Key_13/DOUT
- net Net-(LED14-DOUT) renamed /Key_14/DOUT
- net Net-(LED15-DOUT) renamed /Key_15/DOUT
- net Net-(LED2-DOUT) renamed /Key_2/DOUT
- net Net-(LED3-DOUT) renamed /Key_3/DOUT
- net Net-(LED33-DOUT) renamed /Key_33/DOUT
- net Net-(LED34-DOUT) renamed /Key_34/DOUT
- net Net-(LED35-DOUT) renamed /Key_35/DOUT
- net Net-(LED36-DOUT) renamed /Key_36/DOUT
- net Net-(LED37-DOUT) renamed /Key_37/DOUT
- net Net-(LED38-DOUT) renamed /Key_38/DOUT
- net Net-(LED39-DOUT) renamed /Key_39/DOUT
- net Net-(LED4-DOUT) renamed /Key_4/DOUT
- net Net-(LED40-DOUT) renamed /Key_40/DOUT
- net Net-(LED41-DOUT) renamed /Key_41/DOUT
- net Net-(LED42-DOUT) renamed /Key_42/DOUT
- net Net-(LED43-DOUT) renamed /Key_43/DOUT
- net Net-(LED44-DOUT) renamed /Key_44/DOUT
- net Net-(LED45-DOUT) renamed /Key_45/DOUT
- net Net-(LED46-DOUT) renamed /Key_46/DOUT
- net Net-(LED47-DOUT) renamed /Key_47/DOUT
- net Net-(LED8-DOUT) renamed /Key_8/DOUT
- C1 pad 2: +3.3VD -> +3.3VA
- C10 pad 1: GND -> +3.3VD
- C10 pad 2: Net-(U1-PH1) -> GND
- C11 pad 2: Net-(U1-VCAP_1) -> Net-(U4-NRST)
- C12 pad 2: Net-(U1-VCAP_2) -> Net-(U4-PH0)
- C13 pad 2: +3.3VA -> Net-(U4-PH1)
- C14 pad 1: +3.3VD -> GND
- C14 pad 2: GND -> Net-(U4-VCAP_1)
- C15 pad 2: +5V -> Net-(U4-VCAP_2)
- C16 pad 2: Net-(U2-NR) -> +3.3VA
- C17 pad 1: +3.3VA -> +3.3VD
- C19 pad 2: Net-(U3-NR) -> Net-(U5-NR)
- C2 pad 2: +3.3VD -> Net-(U1D-+)
- C20 pad 1: GND -> +3.3VA
- C20 pad 2: +3.3VA -> GND
- C21 pad 2: +3.3VA -> +5V
- C22 pad 2: +3.3VA -> Net-(U6-NR)
- C3 pad 2: +3.3VD -> +3.3VA
- C6 pad 2: +3.3VA -> +3.3VD
- C7 pad 1: +3.3VD -> GND
- C7 pad 2: GND -> +3.3VD
- C8 pad 2: Net-(U1-NRST) -> +3.3VD
- C9 pad 2: Net-(U1-PH0) -> +3.3VA
- LED1 pad 1: +5V -> Net-(LED1-VDD)
- LED1 pad 3: Net-(LED1-DIN) -> /Key_1/DIN
- LED10 pad 1: +5V -> Net-(LED10-VDD)
- LED11 pad 1: +5V -> Net-(LED11-VDD)
- LED12 pad 1: +5V -> Net-(LED12-VDD)
- LED13 pad 1: +5V -> Net-(LED13-VDD)
- LED14 pad 1: +5V -> Net-(LED14-VDD)
- LED15 pad 1: +5V -> Net-(LED15-VDD)
- LED16 pad 1: +5V -> Net-(LED16-VDD)
- LED16 pad 2: Net-(LED16-DOUT) -> /Key_16/DOUT
- LED17 pad 1: +5V -> Net-(LED17-VDD)
- LED17 pad 2: Net-(LED17-DOUT) -> /Key_17/DOUT
- LED17 pad 3: Net-(LED17-DIN) -> /Key_16/DOUT
- LED18 pad 1: +5V -> Net-(LED18-VDD)
- LED18 pad 2: Net-(LED17-DIN) -> /Key_18/DOUT
- LED18 pad 3: Net-(LED18-DIN) -> /Key_17/DOUT
- LED19 pad 1: +5V -> Net-(LED19-VDD)
- LED19 pad 2: Net-(LED18-DIN) -> /Key_19/DOUT
- LED19 pad 3: Net-(LED19-DIN) -> /Key_18/DOUT
- LED2 pad 1: +5V -> Net-(LED2-VDD)
- LED20 pad 1: +5V -> Net-(LED20-VDD)
- LED20 pad 2: Net-(LED19-DIN) -> /Key_20/DOUT
- LED20 pad 3: Net-(LED20-DIN) -> /Key_19/DOUT
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Routing:
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Other:
- copper layers 4 -> 6
