File: pcb/prometheus-65.kicad_sch (KiCad schematic)
At the start: 65 parts, among them SW1 RotaryEncoder_Switch

Commit message: feat: working changes
Parts:
- removed S1, S10, S12, S13, S17, S18, S19, S2, S20, S21, S22, S23, S24, S25, S26, S27, S28, S29, S3, S30, S31, S33, S34, S35, S36, S37, S38, S39, S4, S40, S41, S42, S43, S44, S45, S46, S47, S49, S50, S51, S53, S54, S55, S58, S6, S60, S64, S7, S9: ~, ScottoKeebs_Hotswap:Hotswap_MX_Plated_1.00u, symbol ScottoKeebs:Placeholder_Keyswitch
- removed S11, S57: ~, ScottoKeebs_Hotswap:Hotswap_MX_Plated_2.25u, symbol ScottoKeebs:Placeholder_Keyswitch
- removed S14, S15, S16, S48, S61, S62, S63: ~, ScottoKeebs_Hotswap:Hotswap_MX_Plated_1.25u, symbol ScottoKeebs:Placeholder_Keyswitch
- removed S32: ~, ScottoKeebs_Hotswap:Hotswap_MX_Plated_6.25u, symbol ScottoKeebs:Placeholder_Keyswitch
- removed S5, S56: ~, ScottoKeebs_Hotswap:Hotswap_MX_Plated_1.50u, symbol ScottoKeebs:Placeholder_Keyswitch
- removed S52: ~, ScottoKeebs_Hotswap:Hotswap_MX_Plated_2.00u, symbol ScottoKeebs:Placeholder_Keyswitch
- removed S59: ~, ScottoKeebs_Hotswap:Hotswap_MX_Plated_2.75u, symbol ScottoKeebs:Placeholder_Keyswitch
- removed S8: ~, ScottoKeebs_Hotswap:Hotswap_MX_Plated_1.75u, symbol ScottoKeebs:Placeholder_Keyswitch
- added C1, C2, C3: 100nF, Capacitor_SMD:C_0402_1005Metric, symbol Device:C
- added J1: Conn_01x04_Socket, Connector_JST:JST_GH_SM04B-GHS-TB_1x04-1MP_P1.25mm_Horizontal, symbol Connector:Conn_01x04_Socket
- added R1, R2: 22Ω, Resistor_SMD:R_0603_1608Metric, symbol Device:R
- added R10, R12, R14, R17, R19, R21, R23, R25, R27, R29, R31, R32, R33, R4, R6, R8: 10kΩ, symbol ScottoKeebs:Placeholder_Resistor
- added R11, R13, R16, R18, R20, R22, R24, R26, R28, R3, R30, R5, R7, R9: 33kΩ, symbol ScottoKeebs:Placeholder_Resistor
- added R15: 330Ω, Resistor_SMD:R_0603_1608Metric, symbol Device:R
- added U1, U2: OPA4323, symbol prometheus-65-symbols:OPA4323
- added U3: 74AHCT125, prometheus-65-footprints:SN74AUC08RGYRG4, symbol 74xx:74AHCT125
Connections:
- net GND: now also C1.1, C2.1, C3.1, J1.4 (Pin_4), R33.1, U1.11 (V-), U2.11 (V-), U3.1, U3.10, U3.12, U3.13, U3.4, U3.5, U3.7 (GND), U3.9
- new net: R11.1, R12.2, U2.10 (+)
- new net: R13.2, R14.2, U2.9 (-)
- new net: R18.2, R19.2, U2.13 (-)
- new net: J1.3 (Pin_3), R2.1
- new net: R30.2, R31.2, U1.9 (-)
- new net: R10.2, R9.2, U2.6 (-)
- new net: R20.1, R21.2, U2.3 (+)
- new net: J1.2 (Pin_2), R1.1
- new net: R28.1, R29.2, U1.10 (+)
- new net: C2.2, R32.2, R33.2, U1.12 (+)
- new net: R5.2, R6.2, U1.2 (-)
- new net: R3.1, R4.2, U1.3 (+)
- new net: R26.2, R27.2, U1.6 (-)
- new net: R22.2, R23.2, U2.2 (-)
- new net: R7.1, R8.2, U2.5 (+)
- new net: R15.1, U3.3
- new net: R16.1, R17.2, U2.12 (+)
- new net: R24.1, R25.2, U1.5 (+)
- new net +1.65VA: R11.2, R16.2, R20.2, R24.2, R28.2, R3.2, R7.2, U1.13 (-), U1.14
- new net +3.3VA: C1.2, C3.2, R32.1, U1.4 (V+), U2.4 (V+)
- new net +5V: J1.1 (Pin_1), U3.14 (VCC)
- new net D+: R2.2
- new net D-: R1.2
- new net Key_84/DOUT: R15.2
- new net Mux_1/MUX_DA: R4.1
- new net Mux_1/MUX_DB: R6.1
- new net Mux_10/MUX_DA: R12.1
- new net Mux_10/MUX_DB: R14.1
- new net Mux_11/MUX_DA: R17.1
- new net Mux_11/MUX_DB: R19.1
- new net Mux_12/MUX_DA: R21.1
- new net Mux_12/MUX_DB: R23.1
- new net Mux_13/MUX_DA: R25.1
- new net Mux_13/MUX_DB: R27.1
- new net Mux_14/MUX_DA: R29.1
- new net Mux_14/MUX_DB: R31.1
- new net Mux_16/MUX_DA: R8.1
- new net Mux_16/MUX_DB: R10.1
- new net STM32F405RGT6/LED_DOUT: U3.2
- new net STM32F405RGT6/MUX_C0: R5.1, U1.1
- new net STM32F405RGT6/MUX_C1: R9.1, U2.7
- new net STM32F405RGT6/MUX_C2: R13.1, U2.8
- new net STM32F405RGT6/MUX_C3: R18.1, U2.14
- new net STM32F405RGT6/MUX_C4: R22.1, U2.1
- new net STM32F405RGT6/MUX_C5: R26.1, U1.7
- new net STM32F405RGT6/MUX_C6: R30.1, U1.8
- no-connect marks 0 -> 4
Other:
- removed sheet LEDs
- removed sheet Mux_0
- removed sheet Power
- removed sheet TMR_0
- removed sheet TMR_1
- removed sheet TMR_10
- removed sheet TMR_11
- removed sheet TMR_12
- removed sheet TMR_13
- removed sheet TMR_14
- removed sheet TMR_15
- removed sheet TMR_16
- removed sheet TMR_17
- removed sheet TMR_18
- removed sheet TMR_19
- removed sheet TMR_2
- removed sheet TMR_20
- removed sheet TMR_21
- removed sheet TMR_22
- removed sheet TMR_23
- removed sheet TMR_24
- removed sheet TMR_25
- removed sheet TMR_26
- removed sheet TMR_27
- removed sheet TMR_28
- removed sheet TMR_29
- removed sheet TMR_3
- removed sheet TMR_30
- removed sheet TMR_31
- removed sheet TMR_32
- removed sheet TMR_33
- removed sheet TMR_34
- removed sheet TMR_35
- removed sheet TMR_36
- removed sheet TMR_37
- removed sheet TMR_38
- removed sheet TMR_39
- removed sheet TMR_4
- removed sheet TMR_40
- removed sheet TMR_41
- removed sheet TMR_42
- removed sheet TMR_43
- removed sheet TMR_44
- removed sheet TMR_45
- removed sheet TMR_46
- removed sheet TMR_47
- removed sheet TMR_48
- removed sheet TMR_49
- removed sheet TMR_5
- removed sheet TMR_50
- removed sheet TMR_51
- removed sheet TMR_52
- removed sheet TMR_53
- removed sheet TMR_54
- removed sheet TMR_55
- removed sheet TMR_56
- removed sheet TMR_57
- removed sheet TMR_58
- removed sheet TMR_59
- removed sheet TMR_6
- removed sheet TMR_60
- removed sheet TMR_61
- removed sheet TMR_62
- removed sheet TMR_63
- removed sheet TMR_7
- removed sheet TMR_8
- removed sheet TMR_9
- added sheet Key_1 (Key.kicad_sch)
- added sheet Key_10 (Key.kicad_sch)
- added sheet Key_11 (Key.kicad_sch)
- added sheet Key_12 (Key.kicad_sch)
- added sheet Key_13 (Key.kicad_sch)
- added sheet Key_14 (Key.kicad_sch)
- added sheet Key_15 (Key.kicad_sch)
- added sheet Key_16 (Key.kicad_sch)
- added sheet Key_17 (Key.kicad_sch)
- added sheet Key_18 (Key.kicad_sch)
- added sheet Key_19 (Key.kicad_sch)
- added sheet Key_2 (Key.kicad_sch)
- added sheet Key_20 (Key.kicad_sch)
- added sheet Key_21 (Key.kicad_sch)
- added sheet Key_22 (Key.kicad_sch)
- added sheet Key_23 (Key.kicad_sch)
- added sheet Key_24 (Key.kicad_sch)
- added sheet Key_25 (Key.kicad_sch)
- added sheet Key_26 (Key.kicad_sch)
- added sheet Key_27 (Key.kicad_sch)
- added sheet Key_28 (Key.kicad_sch)
- added sheet Key_29 (Key.kicad_sch)
- added sheet Key_3 (Key.kicad_sch)
- added sheet Key_30 (Key.kicad_sch)
- added sheet Key_31 (Key.kicad_sch)
- added sheet Key_32 (Key.kicad_sch)
- added sheet Key_33 (Key.kicad_sch)
- added sheet Key_34 (Key.kicad_sch)
- added sheet Key_35 (Key.kicad_sch)
- added sheet Key_36 (Key.kicad_sch)
- added sheet Key_37 (Key.kicad_sch)
- added sheet Key_38 (Key.kicad_sch)
- added sheet Key_39 (Key.kicad_sch)
- added sheet Key_4 (Key.kicad_sch)
- added sheet Key_40 (Key.kicad_sch)
- added sheet Key_41 (Key.kicad_sch)
- added sheet Key_42 (Key.kicad_sch)
- added sheet Key_43 (Key.kicad_sch)
- added sheet Key_44 (Key.kicad_sch)
- added sheet Key_45 (Key.kicad_sch)
- added sheet Key_46 (Key.kicad_sch)
- added sheet Key_47 (Key.kicad_sch)
- added sheet Key_48 (Key.kicad_sch)
- added sheet Key_49 (Key.kicad_sch)
- added sheet Key_5 (Key.kicad_sch)
- added sheet Key_50 (Key.kicad_sch)
- added sheet Key_51 (Key.kicad_sch)
- added sheet Key_52 (Key.kicad_sch)
- added sheet Key_53 (Key.kicad_sch)
- added sheet Key_54 (Key.kicad_sch)
- added sheet Key_55 (Key.kicad_sch)
- added sheet Key_56 (Key.kicad_sch)
- added sheet Key_57 (Key.kicad_sch)
- added sheet Key_58 (Key.kicad_sch)
- added sheet Key_59 (Key.kicad_sch)
- added sheet Key_6 (Key.kicad_sch)
- added sheet Key_60 (Key.kicad_sch)
- added sheet Key_61 (Key.kicad_sch)
- added sheet Key_62 (Key.kicad_sch)
- added sheet Key_63 (Key.kicad_sch)
- added sheet Key_64 (Key.kicad_sch)
- added sheet Key_65 (Key.kicad_sch)
- added sheet Key_66 (Key.kicad_sch)
- added sheet Key_67 (Key.kicad_sch)
- added sheet Key_68 (Key.kicad_sch)
- added sheet Key_69 (Key.kicad_sch)
- added sheet Key_7 (Key.kicad_sch)
- added sheet Key_70 (Key.kicad_sch)
- added sheet Key_71 (Key.kicad_sch)
- added sheet Key_72 (Key.kicad_sch)
- added sheet Key_73 (Key.kicad_sch)
- added sheet Key_74 (Key.kicad_sch)
- added sheet Key_75 (Key.kicad_sch)
- added sheet Key_76 (Key.kicad_sch)
- added sheet Key_77 (Key.kicad_sch)
- added sheet Key_78 (Key.kicad_sch)
- added sheet Key_79 (Key.kicad_sch)
- added sheet Key_8 (Key.kicad_sch)
- added sheet Key_80 (Key.kicad_sch)
- added sheet Key_81 (Key.kicad_sch)
- added sheet Key_82 (Key.kicad_sch)
- added sheet Key_83 (Key.kicad_sch)
- added sheet Key_84 (Key.kicad_sch)
- added sheet Key_9 (Key.kicad_sch)
- added sheet Mux_10 (Multiplexer.kicad_sch)
- added sheet Mux_11 (Multiplexer.kicad_sch)
- added sheet Mux_12 (Multiplexer.kicad_sch)
- added sheet Mux_13 (Multiplexer.kicad_sch)
- added sheet Mux_14 (Multiplexer.kicad_sch)
- added sheet Mux_15 (Multiplexer.kicad_sch)
- added sheet Mux_16 (Multiplexer.kicad_sch)
- added sheet Mux_17 (Multiplexer.kicad_sch)
- added sheet Mux_18 (Multiplexer.kicad_sch)
- added sheet Mux_19 (Multiplexer.kicad_sch)
- added sheet Mux_20 (Multiplexer.kicad_sch)
- added sheet Mux_21 (Multiplexer.kicad_sch)
- added sheet Mux_8 (Multiplexer.kicad_sch)
- added sheet Mux_9 (Multiplexer.kicad_sch)
- added sheet TPS7A4700_A (LDO.kicad_sch)
- added sheet TPS7A4700_D (LDO.kicad_sch)
- sheet Mux_1 ports: added MUX_DA, MUX_DB, MUX_EN, SIG_1A, SIG_1B, SIG_2A, SIG_2B, SIG_3A, SIG_3B, SIG_4A, SIG_4B; removed MUX_D, SIG_0, SIG_1, SIG_2, SIG_3, SIG_4, SIG_5, SIG_6, SIG_7
- sheet Mux_2 ports: added MUX_DA, MUX_DB, MUX_EN, SIG_1A, SIG_1B, SIG_2A, SIG_2B, SIG_3A, SIG_3B, SIG_4A, SIG_4B; removed MUX_D, SIG_0, SIG_1, SIG_2, SIG_3, SIG_4, SIG_5, SIG_6, SIG_7
- sheet Mux_3 ports: added MUX_DA, MUX_DB, MUX_EN, SIG_1A, SIG_1B, SIG_2A, SIG_2B, SIG_3A, SIG_3B, SIG_4A, SIG_4B; removed MUX_D, SIG_0, SIG_1, SIG_2, SIG_3, SIG_4, SIG_5, SIG_6, SIG_7
- sheet Mux_4 ports: added MUX_DA, MUX_DB, MUX_EN, SIG_1A, SIG_1B, SIG_2A, SIG_2B, SIG_3A, SIG_3B, SIG_4A, SIG_4B; removed MUX_D, SIG_0, SIG_1, SIG_2, SIG_3, SIG_4, SIG_5, SIG_6, SIG_7
- sheet Mux_5 ports: added MUX_DA, MUX_DB, MUX_EN, SIG_1A, SIG_1B, SIG_2A, SIG_2B, SIG_3A, SIG_3B, SIG_4A, SIG_4B; removed MUX_D, SIG_0, SIG_1, SIG_2, SIG_3, SIG_4, SIG_5, SIG_6, SIG_7
- sheet Mux_6 ports: added MUX_DA, MUX_DB, MUX_EN, SIG_1A, SIG_1B, SIG_2A, SIG_2B, SIG_3A, SIG_3B, SIG_4A, SIG_4B; removed MUX_D, SIG_0, SIG_1, SIG_2, SIG_3, SIG_4, SIG_5, SIG_6, SIG_7
- sheet Mux_7 ports: added MUX_DA, MUX_DB, MUX_EN, SIG_1A, SIG_1B, SIG_2A, SIG_2B, SIG_3A, SIG_3B, SIG_4A, SIG_4B; removed MUX_D, SIG_0, SIG_1, SIG_2, SIG_3, SIG_4, SIG_5, SIG_6, SIG_7
- sheet STM32F405RGT6: file STM32F405RGT6.kicad_sch -> Microcontroller.kicad_sch
- sheet STM32F405RGT6 ports: added MUX_C0, MUX_C1, MUX_C2, MUX_C3, MUX_C4, MUX_C5, MUX_C6, MUX_EN1, MUX_EN2, MUX_EN3; removed MUX_D0, MUX_D1, MUX_D2, MUX_D3, MUX_D4, MUX_D5, MUX_D6, MUX_D7
- moved on the sheet: SW1
