File: pcb/prometheus-65.kicad_sch (KiCad schematic)
At the start: 65 parts, among them SW1 RotaryEncoder_Switch

Commit message: E
Parts:
- added U77: TMR2615x, prometheus-65-footprints:DFN3L(1.6x1.6x0.5), symbol prometheus-65-symbols:TMR2615x
- S1, S10, S11, S12, S13, S14, S15, S16, S17, S18, S19, S2, S20, S21, S22, S23, S24, S25, S26, S27, S28, S29, S3, S30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: value ~ -> (none)
Connections:
- net GND: now also U77.2 (GND), U77.4 (GND)
